Commit message: funker??

File: src/qube_description/urdf/qube.macro.xacro (robot description, xacro)
@@ -47,10 +47,10 @@
         </link>
         <!-- Joints -->
-        <joint name="${prefix}stator_joint" type="fixed">
+        <joint name="${prefix}base_joint" type="fixed">
             <parent link="${prefix}base_link"/>
             <child link="${prefix}stator_link"/>
             <origin xyz="0 0 ${stator_size/2}" rpy="0 0 0"/>
         </joint>
-        <joint name="${prefix}angle" type="revolute">
+        <joint name="${prefix}motor_joint" type="revolute">
             <parent link="${prefix}stator_link"/>
             <child link="${prefix}rotor_link"/>
@@ -59,5 +59,5 @@
             <limit lower="-3.14159" upper="3.14159" effort="1.0" velocity="1.0"/>
         </joint>
-        <joint name="${prefix}indicator" type="fixed">
+        <joint name="${prefix}rotor_joint" type="fixed">
             <parent link="${prefix}rotor_link"/>
             <child link="${prefix}angle_link"/>
